Commit message: Line_bot complete

File: src/line_bot_description/urdf/robot.urdf (robot description, URDF)
Before this commit: robot line_bot, 5 links, 4 joints
Links:
- added link caster_rear, mass 0.01; collision sphere radius=0.01; visual sphere radius=0.01
Joints:
- added joint caster_rear_joint: type fixed, parent base_link, child caster_rear, origin xyz=-0.055 0 -0.015
